File: STM32_01_PCB.kicad_sch (KiCad schematic)
At the start: 12 parts, among them U1 STM32F411CEUx, Y1 24MHz

Commit message: Add MPU6050
Parts:
- added C10, C11: 100n, symbol Device:C
- added C12: 2n, symbol Device:C
- added C13: 10n, symbol Device:C
- added U2: MPU-6050, Sensor_Motion:InvenSense_QFN-24_4x4mm_P0.5mm, symbol Sensor_Motion:MPU-6050
Connections:
- net +3.3V: now also C10.1, C13.2, U2.13 (VDD), U2.8 (VLOGIC)
- net GND: now also C8.2, C9.2, C10.2, C11.2, C12.2, C13.1, U2.1 (CLKIN), U2.11 (FSYNC), U2.18 (GND)
- new net: C11.1, U2.10 (REGOUT)
- new net: C12.1, U2.20 (CPOUT)

Commit message: USB Input and LDO
Parts:
- added C14, C15: 2n, symbol Device:C
- added C16: 22u, Capacitor_SMD:C_0805_2012Metric_Pad1.18x1.45mm_HandSolder, symbol Device:C
- added D1: LED, symbol Device:LED
- added FB1: 120, symbol Device:FerriteBead
- added J1: USB_B_Micro, symbol Connector:USB_B_Micro
- added R2: 560, symbol Device:R
- added U3: AMS1117-3.3, Package_TO_SOT_SMD:SOT-223-3_TabPin2, symbol Regulator_Linear:AMS1117-3.3
Connections:
- net +3.3V: now also C16.1, D1.2 (A), U3.2 (VO)
- net GND: now also U2.9 (AD0), C14.2, C15.2, C16.2, J1.5 (GND), J1.SH (Shield), R2.2, U3.1 (GND)
- new net +5V: C15.1, FB1.2, U3.3 (VI)
- new net LED_PWR_K: D1.1 (K), R2.1
- new net USB_D+: J1.3 (D+)
- new net USB_D-: J1.2 (D-)
- new net VCC: C14.1, FB1.1, J1.1 (VBUS)
- no-connect marks 0 -> 3
Other:
- moved on the sheet: C1, C10, C11, C12, C13, C2, C3, C4, C5, C6, C7, C8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
